Commit message: XML file is almost prepared. Sensors, actuator were added

File: src/assets/strirus_gamma_30deg_120btw.urdf (robot description, URDF)
Before this commit: robot strirus_gamma, 17 links, 16 joints
Joints:
- joint segment_side_revolute: limit lower=0 upper=0 effort=5 velocity=0.5 -> lower=-0.261799387799 upper=0.261799387799 effort=5 velocity=0.5
- joint segment_up_revolute: limit lower=0 upper=0 effort=5 velocity=0.5 -> lower=-1.308996939 upper=1.308996939 effort=5 velocity=0.5
